File: Breadboard Power Supply/Breadboard Power Supply.kicad_pcb (KiCad board)
At the start: 2 copper layers, 34.5 x 53.6 mm, 19 parts, among them J1 Conn_01x02_Pin, J2 Conn_01x02_Pin, J3 Conn_01x03_Pin, J4 Conn_01x03_Pin, J5 Screw_Terminal_01x02, J6 Barrel_Jack_Switch, J7 Screw_Terminal_01x02, U1 LM7805_TO220, U2 LM317_TO-220

Commit message: update
Parts:
- U1: value LM7805_TO220 -> LM7805
- U2: value LM317_TO-220 -> LM317
- moved U1 4.46 mm to (123.2, 75.9), turned to 0 degrees
Connections:
- J1 pad 2: /PWR_output -> /PWR_OUT_TOP
- J2 pad 2: /PWR_output -> /PWR_OUT_BOT
- J3 pad 2: /PWR_output -> /PWR_OUT_TOP
- J4 pad 2: /PWR_output -> /PWR_OUT_BOT
- J5 pad 2: /PWR_output -> /PWR_OUT_TOP
- J7 pad 2: /PWR_output -> /PWR_OUT_BOT
Routing:
- net /PWR_output: track 128.8 -> 0.00 mm
- net /PWR_OUT_TOP: track 0.00 -> 31.6 mm
- net /PWR_OUT_BOT: track 0.00 -> 28.8 mm
- net /5V: track 68.0 -> 77.1 mm
- net GND: track 10.0 -> 3.42 mm
