File: Breadboard Power Supply/Breadboard Power Supply.kicad_sch (KiCad schematic)
At the start: 17 parts, among them J1 Conn_01x02_Pin, J2 Conn_01x02_Pin, J3 Conn_01x03_Pin, J4 Conn_01x03_Pin, J5 Screw_Terminal_01x02, J6 Barrel_Jack_Switch, J7 Screw_Terminal_01x02, U1 LM7805_TO220, U2 LM317_TO-220

Commit message: update
Connections:
- net PWR_output renamed PWR_OUT_BOT
- net PWR_OUT_BOT: no longer J1.2 (Pin_2), J3.2 (Pin_2), J5.2 (Pin_2)
- new net PWR_OUT_TOP: J1.2 (Pin_2), J3.2 (Pin_2), J5.2 (Pin_2)
Changed lines of the file:
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@@
 	)
 	(rectangle
-		(start 180.34 50.8)
+		(start 179.07 50.8)
 		(end 228.6 142.24)
 		(stroke
@@
 		)
 	)
-	(label "PWR_output"
-		(at 193.04 110.49 180)
-		(effects
-			(font
-				(size 1.27 1.27)
-			)
-			(justify right bottom)
-		)
-	)
 	(label "5V"
 		(at 140.97 50.8 0)
@@
 		)
 	)
+	(label "PWR_OUT_TOP"
+		(at 193.04 63.5 180)
+		(effects
+			(font
+				(size 1.27 1.27)
+			)
+			(justify right bottom)
+		)
+	)
 	(label "PWR_input"
 		(at 69.85 53.34 0)
@@
 		)
 	)
-	(label "PWR_output"
-		(at 193.04 63.5 180)
-		(effects
-			(font
+	(label "PWR_OUT_BOT"
+		(at 193.04 109.22 180)
+		(effects
+			(font
