File: Tiny Solar Supply/Tiny Solar Supply.kicad_pcb (KiCad board)
At the start: 2 copper layers, 38.4 x 22.1 mm, 18 parts, among them J1 Conn_01x02_Pin, J2 Conn_01x02_Pin, J3 Conn_01x02_Pin, J4 Conn_01x02_Pin, Q1 2N7002, U1 AP3015

Commit message: update
Parts:
- moved L1 0.13 mm to (102.1, 90.8)
Routing:
- net Net-(J3-Pin_1): track 33.1 -> 34.8 mm
